File: Electronics/Battey Spacer 1/BatterySpacer1.brd (EAGLE design)
At the start: 30 x 30 mm, 0 parts

Commit message: connector PCBs and such
Other:
- board size 30 x 30 mm -> 28.5 x 28.5 mm
Changed lines of the file:
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@@
 <circle x="14" y="14" radius="14.25" width="0.01" layer="20"/>
 <circle x="14" y="14" radius="8" width="0.01" layer="20"/>
-<wire x1="4" y1="17" x2="4" y2="11" width="0.01" layer="20"/>
-<wire x1="24" y1="17" x2="24" y2="11" width="0.01" layer="20"/>
 <wire x1="4.625" y1="17" x2="4.625" y2="11" width="0.01" layer="20"/>
 <wire x1="3.375" y1="17" x2="3.375" y2="11" width="0.01" layer="20"/>
@@
 <wire x1="3.375" y1="17" x2="4.625" y2="17" width="0.01" layer="20" curve="-180"/>
 <wire x1="4.625" y1="11" x2="3.375" y2="11" width="0.01" layer="20" curve="-180"/>
-<wire x1="-1" y1="14" x2="14" y2="14" width="0.01" layer="20"/>
-<wire x1="14" y1="14" x2="29" y2="14" width="0.01" layer="20"/>
-<wire x1="14" y1="29" x2="14" y2="14" width="0.01" layer="20"/>
-<wire x1="14" y1="14" x2="14" y2="-1" width="0.01" layer="20"/>
-<wire x1="14" y1="14" x2="3" y2="25" width="0.01" layer="20"/>
-<wire x1="14" y1="14" x2="25" y2="25" width="0.01" layer="20"/>
-<wire x1="14" y1="14" x2="26" y2="2" width="0.01" layer="20"/>
-<wire x1="14" y1="14" x2="3" y2="3" width="0.01" layer="20"/>
 </plain>
 <attributes>

Commit message: pcb spacer and breakoutoard over
Routing:
- net BAT: track 0.00 -> 82.7 mm, vias 0 -> 67
- net N$70: track 4.00 -> 0.00 mm, vias 2 -> 0
- added copper zone on layer 1, net BAT
- added copper zone on layer 16, net BAT
Other:
- outline, holes or cut-outs redrawn
