File: Electronics/Business Card/BotSide.brd (EAGLE design)
At the start: 85 x 50 mm, 0 parts

Commit message: connector PCBs and such
Changed lines of the file:
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@@
 <layer number="27" name="tValues" color="7" fill="1" visible="yes" active="yes"/>
 <layer number="28" name="bValues" color="7" fill="1" visible="yes" active="yes"/>
-<layer number="29" name="tStop" color="7" fill="3" visible="no" active="yes"/>
+<layer number="29" name="tStop" color="7" fill="3" visible="yes" active="yes"/>
 <layer number="30" name="bStop" color="7" fill="6" visible="no" active="yes"/>
 <layer number="31" name="tCream" color="7" fill="4" visible="no" active="yes"/>
@@
 <layer number="43" name="vRestrict" color="2" fill="10" visible="yes" active="yes"/>
 <layer number="44" name="Drills" color="7" fill="1" visible="no" active="yes"/>
-<layer number="45" name="Holes" color="7" fill="1" visible="no" active="yes"/>
+<layer number="45" name="Holes" color="7" fill="1" visible="yes" active="yes"/>
 <layer number="46" name="Milling" color="3" fill="1" visible="no" active="yes"/>
 <layer number="47" name="Measures" color="7" fill="1" visible="no" active="yes"/>
@@
 <wire x1="85" y1="5" x2="80" y2="0" width="0.01" layer="20" curve="-90"/>
 <wire x1="5" y1="0" x2="0" y2="5" width="0.01" layer="20" curve="-90"/>
-<text x="5" y="40" size="5" layer="25" font="fixed">Daniil Andreev</text>
-<text x="5" y="35" size="4" layer="25" font="fixed">Hardware Engineer</text>
-<text x="5" y="19" size="3" layer="25" font="fixed">dannyandreev.com</text>
-<text x="5" y="25" size="3" layer="25" font="fixed">650-704-9677</text>
-<text x="5" y="29" size="3" layer="25" font="fixed">andreev.danny@gmail.com</text>
-<circle x="20" y="5" radius="0.1" width="0.4" layer="17"/>
-<circle x="25" y="10" radius="0.1" width="0.4" layer="17"/>
-<circle x="15" y="5" radius="0.1" width="0.4" layer="17"/>
-<circle x="10" y="5" radius="0.1" width="0.4" layer="17"/>
-<circle x="15" y="10" radius="0.1" width="0.4" layer="17"/>
-<circle x="20" y="10" radius="0.1" width="0.4" layer="17"/>
-<circle x="20" y="15" radius="0.1" width="0.4" layer="17"/>
-<circle x="25" y="15" radius="0.1" width="0.4" layer="17"/>
-<circle x="30" y="15" radius="0.1" width="0.4" layer="17"/>
-<circle x="40" y="25" radius="0.1" width="0.4" layer="17"/>
-<circle x="35" y="25" radius="0.1" width="0.4" layer="17"/>
-<circle x="60" y="45" radius="0.1" width="0.4" layer="17"/>
-<circle x="55" y="45" radius="0.1" width="0.4" layer="17"/>
-<circle x="50" y="45" radius="0.1" width="0.4" layer="17"/>
+<text x="5" y="39" size="5.5" layer="25" font="fixed">Daniil Andreev</text>
+<text x="5" y="34" size="4.2" layer="25" font="fixed">Hardware Engineer</text>
+<text x="5" y="17" size="2.48" layer="25" font="fixed">dannyandreev.com</text>
+<text x="5" y="27" size="2.86" layer="25" font="fixed">andreev.danny@gmail.com</text>
+<text x="5" y="23" size="2.86" layer="25" font="fixed">650-704-9677</text>
 </plain>
 <attributes>
@@
 <signal name="N$55">
 <via x="65" y="40" extent="1-16" drill="0.5"/>
+<via x="60" y="40" extent="1-16" drill="0.5"/>
+<via x="60" y="35" extent="1-16" drill="0.5"/>
+<via x="60" y="30" extent="1-16" drill="0.5"/>
+<via x="55" y="30" extent="1-16" drill="0.5"/>
+<via x="55" y="35" extent="1-16" drill="0.5"/>
+<via x="50" y="30" extent="1-16" drill="0.5"/>
+<wire x1="60" y1="40" x2="65" y2="40" width="0" layer="19" extent="1-1"/>
+<wire x1="60" y1="35" x2="60" y2="40" width="0" layer="19" extent="1-1"/>
+<wire x1="60" y1="30" x2="60" y2="35" width="0" layer="19" extent="1-1"/>
+<wire x1="55" y1="35" x2="60" y2="35" width="0" layer="19" extent="1-1"/>
+<wire x1="55" y1="30" x2="60" y2="30" width="0" layer="19" extent="1-1"/>
+<wire x1="50" y1="30" x2="55" y2="30" width="0" layer="19" extent="1-1"/>
 </signal>
 <signal name="N$56">
@@
 <via x="50" y="25" extent="1-16" drill="0.5"/>
 </signal>
+<signal name="N$77">
+<via x="30" y="15" extent="1-16" drill="0.000009375"/>
+</signal>
 <signal name="N$58">
 <via x="45" y="25" extent="1-16" drill="0.5"/>
+<via x="40" y="25" extent="1-16" drill="0.000009375"/>
+<via x="45" y="20" extent="1-16" drill="0.5"/>
+<via x="40" y="20" extent="1-16" drill="0.5"/>
+<via x="35" y="25" extent="1-16" drill="0.000009375"/>
+<wire x1="40" y1="25" x2="45" y2="25" width="0" layer="19" extent="1-1"/>
+<wire x1="45" y1="20" x2="45" y2="25" width="0" layer="19" extent="1-1"/>
+<wire x1="40" y1="20" x2="40" y2="25" width="0" layer="19" extent="1-1"/>
+<wire x1="35" y1="25" x2="40" y2="25" width="0" layer="19" extent="1-1"/>
 </signal>
 <signal name="N$59">
@@
 <signal name="N$62">
 <via x="35" y="15" extent="1-16" drill="0.5"/>
+<via x="35" y="20" extent="1-16" drill="0.5"/>
+<wire x1="35" y1="15" x2="35" y2="20" width="0" layer="19" extent="1-1"/>
 </signal>
 <signal name="N$63">
@@
 </polygon>
 </signal>
+<signal name="N$66">
+<via x="25" y="15" extent="1-16" drill="0.000009375"/>
+</signal>
+<signal name="N$67">
+<via x="20" y="15" extent="1-16" drill="0.000009375"/>
+</signal>
+<signal name="N$68">
+<via x="20" y="5" extent="1-16" drill="0.000009375"/>
+</signal>
+<signal name="N$69">
+<via x="15" y="5" extent="1-16" drill="0.000009375"/>
+</signal>
+<signal name="N$70">
+<via x="10" y="5" extent="1-16" drill="0.000009375"/>
+</signal>
+<signal name="N$71">
+<via x="20" y="10" extent="1-16" drill="0.000009375"/>
+</signal>
+<signal name="N$72">
+<via x="25" y="10" extent="1-16" drill="0.000009375"/>
+</signal>
+<signal name="N$73">
+<via x="15" y="10" extent="1-16" drill="0.000009375"/>
+</signal>
+<signal name="N$74">
+<via x="60" y="45" extent="1-16" drill="0.000009375"/>
+<via x="55" y="40" extent="1-16" drill="0.000009375"/>
+<via x="50" y="40" extent="1-16" drill="0.000009375"/>
+<via x="50" y="35" extent="1-16" drill="0.000009375"/>
+<wire x1="55" y1="40" x2="60" y2="45" width="0" layer="19" extent="1-1"/>
+<wire x1="50" y1="40" x2="55" y2="40" width="0" layer="19" extent="1-1"/>
+<wire x1="50" y1="35" x2="50" y2="40" width="0" layer="19" extent="1-1"/>
+</signal>
+<signal name="N$75">
+<via x="55" y="45" extent="1-16" drill="0.000009375"/>
+</signal>
+<signal name="N$76">
+<via x="50" y="45" extent="1-16" drill="0.000009375"/>
+</signal>
 </signals>
