File: Electronics/BMS/BMSMAX14921/BMSMAX14921Based.brd (EAGLE design)
At the start: 55.4 x 41.7 mm, 66 parts, among them IC1 MAX14921, J1 CONNECTOR_9PIN, J4 CONNECTOR_9PIN, J5 CONNECTOR_8PIN, J6 CONNECTOR_9PIN

Commit message: dank work bean
Parts:
- added >MOS1, >MOS2: NMOS_IRFS7730, MarkIIEaglelbr:D2PAK-7PIN
- added U$1: ACS758XCB, MarkIIEaglelbr:CB5PFF
- moved IC1 36.1 mm to (33.1, 51.8)
- moved C1 36.0 mm to (35.6, 63.0)
- moved C10 36.0 mm to (21.3, 49.3)
- moved C11 36.0 mm to (21.3, 52.1)
- moved C12 36.0 mm to (21.3, 54.9)
- moved C13 36.0 mm to (21.3, 57.7)
- moved C14 36.0 mm to (27.2, 63.0)
- moved C15 36.0 mm to (30.0, 63.0)
- moved C16 36.0 mm to (32.8, 63.0)
- moved C18 36.0 mm to (33.3, 40.6)
- moved C19 36.0 mm to (31.0, 40.6)
- moved C2 36.0 mm to (38.4, 63.0)
- moved C3 36.0 mm to (43.7, 57.1)
- moved C4 36.0 mm to (43.7, 54.4)
- moved C5 36.0 mm to (43.7, 51.6)
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Routing:
- net VP: track 68.3 -> 0.00 mm, vias 1 -> 0
- net CV1: track 65.2 -> 0.00 mm
- net CV15: track 60.1 -> 0.00 mm
- net CV8: track 55.7 -> 0.00 mm
- net CV7: track 55.3 -> 0.00 mm
- net CV5: track 52.0 -> 0.00 mm
- net CV2: track 50.2 -> 0.00 mm
- net CV14: track 47.9 -> 0.00 mm
- net 3V3: track 43.8 -> 0.00 mm, vias 1 -> 0
- net CV3: track 43.1 -> 0.00 mm
- net CV6: track 39.6 -> 0.00 mm, vias 1 -> 0
- net BA8: track 39.2 -> 0.00 mm
- net CV13: track 38.7 -> 0.00 mm
- net CV4: track 37.1 -> 0.00 mm
- net BA7: track 35.6 -> 0.00 mm
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- removed copper zone on layer 1, net GND
- removed copper zone on layer 16, net GND
Other:
- board size 55.4 x 41.7 mm -> 63.5 x 31.8 mm

Commit message: cleaned up files, created legacy folders
Parts:
- moved J6 40.4 mm to (33.3, 36.7)
- moved J4 27.3 mm to (34.0, 61.7), turned to 0 degrees
- moved J5 16.2 mm to (32.6, 64.6)
- moved J1 11.5 mm to (33.4, 39.5), turned to 0 degrees
- moved IC1 1.02 mm to (33.0, 50.8)
