File: Electronics/PCBEndCap/PCBEndCap.sch (EAGLE design)
At the start: 2 parts, among them J3 CONNECTOR_9PIN, J4 CONNECTOR_9PIN

Commit message: pcb spacer and breakoutoard over
Parts:
- removed J3, J4: CONNECTOR_9PIN, lolomolo:CONNECTOR_9PIN
- added J1: CONNECTORJST2X9_2MM, MarkIIEaglelbr:CONNECTORJST2X9_2MM
Connections:
- removed net N1: J3.P$2
- removed net N10: J4.P$2
- removed net N11: J4.P$3
- removed net N12: J4.P$4
- removed net N13: J4.P$5
- removed net N14: J4.P$6
- removed net N15: J4.P$7
- removed net N16: J4.P$8
- removed net N2: J3.P$3
- removed net N3: J3.P$4
- removed net N4: J3.P$5
- removed net N5: J3.P$6
- removed net N6: J3.P$7
- removed net N7: J3.P$8
- removed net N8: J3.P$9
- removed net N9: J4.P$1
- new net B1: J1.P$2
- new net B10: J1.P$7
- new net B11: J1.P$6
- new net B12: J1.P$14
- new net B13: J1.P$13
- new net B14: J1.P$12
- new net B15: J1.P$11
- new net B16: J1.P$10
- new net B2: J1.P$3
- new net B3: J1.P$4
- new net B4: J1.P$5
- new net B5: J1.P$15
- new net B6: J1.P$16
- new net B7: J1.P$17
- new net B8: J1.P$18
- new net B9: J1.P$8
- net GND: now also J1.P$1; no longer J3.P$1
- net VCC: now also J1.P$9; no longer J4.P$9
Changed lines of the file:
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@@
 </classes>
 <parts>
-<part name="J3" library="lolomolo" deviceset="CONNECTOR_9PIN" device=""/>
-<part name="J4" library="lolomolo" deviceset="CONNECTOR_9PIN" device=""/>
+<part name="J1" library="MarkIIEaglelbr" deviceset="CONNECTORJST2X9_2MM" device=""/>
 </parts>
 <sheets>
@@
 </plain>
 <instances>
-<instance part="J3" gate="G$1" x="66.04" y="73.66" rot="R90"/>
-<instance part="J4" gate="G$1" x="63.5" y="40.64" rot="R270"/>
+<instance part="J1" gate="G$1" x="66.04" y="58.42"/>
 </instances>
 <busses>
 </busses>
 <nets>
-<net name="N1" class="0">
+<net name="B16" class="0">
 <segment>
-<wire x1="58.42" y1="63.5" x2="58.42" y2="60.96" width="0.1524" layer="91"/>
-<pinref part="J3" gate="G$1" pin="P$2"/>
-<label x="58.42" y="63.5" size="1.778" layer="95" rot="R270"/>
+<wire x1="76.2" y1="66.04" x2="76.2" y2="63.5" width="0.1524" layer="91"/>
+<label x="76.2" y="66.04" size="1.778" layer="95" rot="R270"/>
+<pinref part="J1" gate="G$1" pin="P$10"/>
 </segment>
 </net>
-<net name="N2" class="0">
+<net name="B2" class="0">
 <segment>
-<wire x1="60.96" y1="63.5" x2="60.96" y2="60.96" width="0.1524" layer="91"/>
-<pinref part="J3" gate="G$1" pin="P$3"/>
-<label x="60.96" y="63.5" size="1.778" layer="95" rot="R270"/>
+<wire x1="60.96" y1="53.34" x2="60.96" y2="50.8" width="0.1524" layer="91"/>
+<label x="60.96" y="53.34" size="1.778" layer="95" rot="R270"/>
+<pinref part="J1" gate="G$1" pin="P$3"/>
 </segment>
 </net>
-<net name="N3" class="0">
+<net name="B3" class="0">
 <segment>
-<wire x1="63.5" y1="63.5" x2="63.5" y2="60.96" width="0.1524" layer="91"/>
-<pinref part="J3" gate="G$1" pin="P$4"/>
-<label x="63.5" y="63.5" size="1.778" layer="95" rot="R270"/>
+<wire x1="63.5" y1="53.34" x2="63.5" y2="50.8" width="0.1524" layer="91"/>
+<label x="63.5" y="53.34" size="1.778" layer="95" rot="R270"/>
+<pinref part="J1" gate="G$1" pin="P$4"/>
 </segment>
 </net>
-<net name="N4" class="0">
+<net name="B4" class="0">
 <segment>
-<wire x1="66.04" y1="63.5" x2="66.04" y2="60.96" width="0.1524" layer="91"/>
-<pinref part="J3" gate="G$1" pin="P$5"/>
-<label x="66.04" y="63.5" size="1.778" layer="95" rot="R270"/>
+<wire x1="66.04" y1="53.34" x2="66.04" y2="50.8" width="0.1524" layer="91"/>
+<label x="66.04" y="53.34" size="1.778" layer="95" rot="R270"/>
+<pinref part="J1" gate="G$1" pin="P$5"/>
 </segment>
 </net>
-<net name="N5" class="0">
+<net name="B6" class="0">
 <segment>
-<wire x1="68.58" y1="63.5" x2="68.58" y2="60.96" width="0.1524" layer="91"/>
-<pinref part="J3" gate="G$1" pin="P$6"/>
-<label x="68.58" y="63.5" size="1.778" layer="95" rot="R270"/>
+<wire x1="60.96" y1="66.04" x2="60.96" y2="63.5" width="0.1524" layer="91"/>
+<label x="60.96" y="66.04" size="1.778" layer="95" rot="R270"/>
+<pinref part="J1" gate="G$1" pin="P$16"/>
 </segment>
 </net>
-<net name="N6" class="0">
+<net name="B7" class="0">
 <segment>
-<wire x1="71.12" y1="63.5" x2="71.12" y2="60.96" width="0.1524" layer="91"/>
-<pinref part="J3" gate="G$1" pin="P$7"/>
-<label x="71.12" y="63.5" size="1.778" layer="95" rot="R270"/>
+<wire x1="58.42" y1="66.04" x2="58.42" y2="63.5" width="0.1524" layer="91"/>
+<label x="58.42" y="66.04" size="1.778" layer="95" rot="R270"/>
+<pinref part="J1" gate="G$1" pin="P$17"/>
 </segment>
 </net>
-<net name="N7" class="0">
+<net name="B8" class="0">
 <segment>
-<wire x1="73.66" y1="63.5" x2="73.66" y2="60.96" width="0.1524" layer="91"/>
-<pinref part="J3" gate="G$1" pin="P$8"/>
-<label x="73.66" y="63.5" size="1.778" layer="95" rot="R270"/>
+<wire x1="55.88" y1="66.04" x2="55.88" y2="63.5" width="0.1524" layer="91"/>
+<label x="55.88" y="66.04" size="1.778" layer="95" rot="R270"/>
+<pinref part="J1" gate="G$1" pin="P$18"/>
 </segment>
 </net>
-<net name="N8" class="0">
+<net name="B15" class="0">
 <segment>
-<wire x1="76.2" y1="63.5" x2="76.2" y2="60.96" width="0.1524" layer="91"/>
-<pinref part="J3" gate="G$1" pin="P$9"/>
-<label x="76.2" y="63.5" size="1.778" layer="95" rot="R270"/>
-<label x="76.2" y="63.5" size="1.778" layer="95" rot="R270"/>
+<pinref part="J1" gate="G$1" pin="P$11"/>
+<wire x1="73.66" y1="63.5" x2="73.66" y2="66.04" width="0.1524" layer="91"/>
+<label x="73.66" y="66.04" size="1.778" layer="95" rot="R270"/>
 </segment>
 </net>
-<net name="N16" class="0">
+<net name="GND" class="0">
 <segment>
-<wire x1="55.88" y1="53.34" x2="55.88" y2="50.8" width="0.1524" layer="91"/>
-<pinref part="J4" gate="G$1" pin="P$8"/>
+<wire x1="55.88" y1="50.8" x2="55.88" y2="53.34" width="0.1524" layer="91"/>
 <label x="55.88" y="53.34" size="1.778" layer="95" rot="R270"/>
+<pinref part="J1" gate="G$1" pin="P$1"/>
 </segment>
 </net>
-<net name="N15" class="0">
+<net name="B5" class="0">
 <segment>
+<wire x1="63.5" y1="66.04" x2="63.5" y2="63.5" width="0.1524" layer="91"/>
+<label x="63.5" y="66.04" size="1.778" layer="95" rot="R270"/>
+<pinref part="J1" gate="G$1" pin="P$15"/>
+</segment>
+</net>
+<net name="B1" class="0">
+<segment>
+<pinref part="J1" gate="G$1" pin="P$2"/>
 <wire x1="58.42" y1="53.34" x2="58.42" y2="50.8" width="0.1524" layer="91"/>
-<pinref part="J4" gate="G$1" pin="P$7"/>
 <label x="58.42" y="53.34" size="1.778" layer="95" rot="R270"/>
 </segment>
 </net>
-<net name="N14" class="0">
+<net name="B13" class="0">
 <segment>
-<wire x1="60.96" y1="53.34" x2="60.96" y2="50.8" width="0.1524" layer="91"/>
-<pinref part="J4" gate="G$1" pin="P$6"/>
-<label x="60.96" y="53.34" size="1.778" layer="95" rot="R270"/>
+<pinref part="J1" gate="G$1" pin="P$13"/>
+<wire x1="68.58" y1="63.5" x2="68.58" y2="66.04" width="0.1524" layer="91"/>
+<label x="68.58" y="66.04" size="1.778" layer="95" rot="R270"/>
 </segment>
 </net>
-<net name="N13" class="0">
+<net name="B14" class="0">
 <segment>
-<wire x1="63.5" y1="53.34" x2="63.5" y2="50.8" width="0.1524" layer="91"/>
-<pinref part="J4" gate="G$1" pin="P$5"/>
-<label x="63.5" y="53.34" size="1.778" layer="95" rot="R270"/>
+<label x="71.12" y="66.04" size="1.778" layer="95" rot="R270"/>
+<pinref part="J1" gate="G$1" pin="P$12"/>
+<wire x1="71.12" y1="66.04" x2="71.12" y2="63.5" width="0.1524" layer="91"/>
 </segment>
 </net>
-<net name="N12" class="0">
+<net name="B12" class="0">
 <segment>
-<wire x1="66.04" y1="53.34" x2="66.04" y2="50.8" width="0.1524" layer="91"/>
-<pinref part="J4" gate="G$1" pin="P$4"/>
-<label x="66.04" y="53.34" size="1.778" layer="95" rot="R270"/>
-</segment>
-</net>
-<net name="N11" class="0">
-<segment>
-<wire x1="68.58" y1="53.34" x2="68.58" y2="50.8" width="0.1524" layer="91"/>
-<pinref part="J4" gate="G$1" pin="P$3"/>
-<label x="68.58" y="53.34" size="1.778" layer="95" rot="R270"/>
-</segment>
-</net>
-<net name="N10" class="0">
-<segment>
-<wire x1="71.12" y1="53.34" x2="71.12" y2="50.8" width="0.1524" layer="91"/>
-<pinref part="J4" gate="G$1" pin="P$2"/>
-<label x="71.12" y="53.34" size="1.778" layer="95" rot="R270"/>
-</segment>
-</net>
-<net name="N9" class="0">
-<segment>
-<wire x1="73.66" y1="53.34" x2="73.66" y2="50.8" width="0.1524" layer="91"/>
-<pinref part="J4" gate="G$1" pin="P$1"/>
-<label x="73.66" y="53.34" size="1.778" layer="95" rot="R270"/>
+<wire x1="66.04" y1="66.04" x2="66.04" y2="63.5" width="0.1524" layer="91"/>
+<label x="66.04" y="66.04" size="1.778" layer="95" rot="R270"/>
+<pinref part="J1" gate="G$1" pin="P$14"/>
 </segment>
 </net>
 <net name="VCC" class="0">
 <segment>
-<wire x1="53.34" y1="50.8" x2="53.34" y2="53.34" width="0.1524" layer="91"/>
-<pinref part="J4" gate="G$1" pin="P$9"/>
-<label x="53.34" y="53.34" size="1.778" layer="95" rot="R270"/>
+<pinref part="J1" gate="G$1" pin="P$9"/>
+<wire x1="76.2" y1="53.34" x2="76.2" y2="50.8" width="0.1524" layer="91"/>
+<label x="76.2" y="53.34" size="1.778" layer="95" rot="R270"/>
 </segment>
 </net>
-<net name="GND" class="0">
+<net name="B10" class="0">
 <segment>
-<wire x1="55.88" y1="63.5" x2="55.88" y2="60.96" width="0.1524" layer="91"/>
-<pinref part="J3" gate="G$1" pin="P$1"/>
-<label x="55.88" y="63.5" size="1.778" layer="95" rot="R270"/>
+<label x="71.12" y="53.34" size="1.778" layer="95" rot="R270"/>
+<pinref part="J1" gate="G$1" pin="P$7"/>
+<wire x1="71.12" y1="53.34" x2="71.12" y2="50.8" width="0.1524" layer="91"/>
 </segment>
 </net>
+<net name="B9" class="0">
+<segment>
+<pinref part="J1" gate="G$1" pin="P$8"/>
+<wire x1="73.66" y1="53.34" x2="73.66" y2="50.8" width="0.1524" layer="91"/>
+<label x="73.66" y="53.34" size="1.778" layer="95" rot="R270"/>
+</segment>
+</net>
+<net name="B11" class="0">
+<segment>
+<pinref part="J1" gate="G$1" pin="P$6"/>
+<wire x1="68.58" y1="50.8" x2="68.58" y2="53.34" width="0.1524" layer="91"/>
+<label x="68.58" y="53.34" size="1.778" layer="95" rot="R270"/>
+</segment>
+</net>
