File: Electronics/BMS/BMSMAX14921Breakout/BMSMAX14921Based.brd (EAGLE design)
At the start: 55.4 x 41.7 mm, 66 parts, among them IC1 MAX14921, J1 CONNECTOR_9PIN, J4 CONNECTOR_9PIN, J5 CONNECTOR_8PIN, J6 CONNECTOR_9PIN

Commit message: pcb spacer and breakoutoard over
Parts:
- added J2: CONNECTORJST2X9_2MM, MarkIIEaglelbr:CONNECTOR9X2_2MMPITCH
- moved J5 4.32 mm to (15.0, 44.2)
- moved J6 4.32 mm to (39.1, 44.2)
- moved R18 0.40 mm to (29.6, 4.95)
- moved C19 0.13 mm to (25.5, 5.08)
Connections:
- net 3V3: now also IC1.P$5; no longer IC1.5
- net 5V: now also IC1.P$12, IC1.P$13; no longer IC1.12, IC1.13
- net AOUT: now also IC1.P$10; no longer IC1.10
- net BA1: now also IC1.P$76; no longer IC1.76
- net BA10: now also IC1.P$40; no longer IC1.40
- net BA11: now also IC1.P$36; no longer IC1.36
- net BA12: now also IC1.P$32; no longer IC1.32
- net BA13: now also IC1.P$28; no longer IC1.28
- net BA14: now also IC1.P$24; no longer IC1.24
- net BA15: now also IC1.P$20; no longer IC1.20
- net BA16: now also IC1.P$16; no longer IC1.16
- net BA2: now also IC1.P$72; no longer IC1.72
- net BA3: now also IC1.P$68; no longer IC1.68
- net BA4: now also IC1.P$64; no longer IC1.64
- net BA5: now also IC1.P$60; no longer IC1.60
- net BA6: now also IC1.P$56; no longer IC1.56
- net BA7: now also IC1.P$52; no longer IC1.52
- net BA8: now also IC1.P$48; no longer IC1.48
- net BA9: now also IC1.P$44; no longer IC1.44
- net CB10: now also IC1.P$42; no longer IC1.42
- net CB11: now also IC1.P$38; no longer IC1.38
- net CB12: now also IC1.P$34; no longer IC1.34
- net CB13: now also IC1.P$30; no longer IC1.30
- net CB14: now also IC1.P$26; no longer IC1.26
- net CB15: now also IC1.P$22; no longer IC1.22
- net CB16: now also IC1.P$18; no longer IC1.18
- net CB2: now also IC1.P$74; no longer IC1.74
- net CB3: now also IC1.P$70; no longer IC1.70
- net CB4: now also IC1.P$66; no longer IC1.66
- net CB5: now also IC1.P$62; no longer IC1.62
- net CB6: now also IC1.P$58; no longer IC1.58
- net CB7: now also IC1.P$54; no longer IC1.54
- net CB8: now also IC1.P$50; no longer IC1.50
- net CB9: now also IC1.P$46; no longer IC1.46
- net CS: now also IC1.P$80; no longer IC1.80
- net CT1: now also IC1.P$77; no longer IC1.77
- net CT10: now also IC1.P$41; no longer IC1.41
- net CT11: now also IC1.P$37; no longer IC1.37
- net CT12: now also IC1.P$33; no longer IC1.33
- net CT13: now also IC1.P$29; no longer IC1.29
- net CT14: now also IC1.P$25; no longer IC1.25
- net CT15: now also IC1.P$21; no longer IC1.21
- net CT16: now also IC1.P$17; no longer IC1.17
- net CT2: now also IC1.P$73; no longer IC1.73
- net CT3: now also IC1.P$69; no longer IC1.69
- net CT4: now also IC1.P$65; no longer IC1.65
- net CT5: now also IC1.P$61; no longer IC1.61
- net CT6: now also IC1.P$57; no longer IC1.57
- net CT7: now also IC1.P$53; no longer IC1.53
- net CT8: now also IC1.P$49; no longer IC1.49
- net CT9: now also IC1.P$45; no longer IC1.45
- net CV1: now also J2.P$2
- net CV10: now also J2.P$7
- net CV11: now also J2.P$6
- net CV12: now also J2.P$14
- net CV13: now also J2.P$13
- net CV14: now also J2.P$12
- net CV15: now also J2.P$11
- net CV2: now also J2.P$3
- net CV3: now also J2.P$4
- net CV4: now also J2.P$5
- net CV5: now also J2.P$15
- net CV6: now also J2.P$16
- net CV7: now also J2.P$17
- net CV8: now also J2.P$18
- net CV9: now also J2.P$8
- net DGND: now also IC1.P$6; no longer IC1.6
- net EN: now also IC1.P$79; no longer IC1.79
- net GND: now also IC1.P$11, IC1.P$78, J2.P$1; no longer IC1.11, IC1.78
- net N$11: now also IC1.P$67; no longer IC1.67
- net N$12: now also IC1.P$75; no longer IC1.75
- net N$26: now also IC1.P$63; no longer IC1.63
- net N$29: now also IC1.P$59; no longer IC1.59
- net N$30: now also IC1.P$55; no longer IC1.55
- net N$31: now also IC1.P$51; no longer IC1.51
- net N$32: now also IC1.P$47; no longer IC1.47
- net N$33: now also IC1.P$43; no longer IC1.43
- net N$34: now also IC1.P$39; no longer IC1.39
- net N$35: now also IC1.P$35; no longer IC1.35
- net N$36: now also IC1.P$31; no longer IC1.31
- net N$37: now also IC1.P$27; no longer IC1.27
- net N$38: now also IC1.P$23; no longer IC1.23
- net N$39: now also IC1.P$19; no longer IC1.19
- net N$40: now also IC1.P$15; no longer IC1.15
- net N$9: now also IC1.P$71; no longer IC1.71
- net SAMPL: now also IC1.P$4; no longer IC1.4
- net SCLK: now also IC1.P$1; no longer IC1.1
- net SDI: now also IC1.P$2; no longer IC1.2
- net SDO: now also IC1.P$3; no longer IC1.3
- net T1: now also IC1.P$9; no longer IC1.9
- net T2: now also IC1.P$8; no longer IC1.8
- net T3: now also IC1.P$7; no longer IC1.7
- net VP: now also IC1.P$14, J2.P$10, J2.P$9; no longer IC1.14
Routing:
- net CV9: track 26.7 -> 51.6 mm
- net CV11: track 29.9 -> 54.4 mm, vias 0 -> 1
- net CV8: track 55.7 -> 79.1 mm
- net CV10: track 23.4 -> 46.5 mm, vias 0 -> 1
- net CV6: track 39.6 -> 62.2 mm, vias 1 -> 2
- net CV12: track 32.4 -> 53.8 mm
- net CV13: track 38.7 -> 57.4 mm, vias 0 -> 1
- net CV5: track 52.0 -> 70.3 mm
- net CV4: track 37.1 -> 55.4 mm
- net CV7: track 55.3 -> 73.3 mm
- net VP: track 68.3 -> 84.7 mm
- net CV14: track 47.9 -> 62.5 mm, vias 0 -> 1
- net CV3: track 43.1 -> 57.4 mm, vias 0 -> 1
- net CV2: track 50.2 -> 61.6 mm, vias 0 -> 1
- net CV15: track 60.1 -> 70.3 mm, vias 0 -> 1
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Other:
- board size 55.4 x 41.7 mm -> 55.4 x 46.1 mm

Commit message: updated Max14921 Breakout Board
Parts:
- added C20, C22, C25, C27: 1uF, lolomolo:0805_(2012_METRIC)
- added C21, C23, C24, C26: .1uF, lolomolo:0805_(2012_METRIC)
- added IC2: ADC141S626, MarkIIEaglelbr:10-VSSOP
- added R35, R36: 0, lolomolo:0805_(2012_METRIC)
- added V1: (no value), MarkIIEaglelbr:SOT-23
- C19: value 1uF -> .1uF
- moved R1 6.49 mm to (12.1, 5.21), turned to 180 degrees
- moved R18 2.25 mm to (28.1, 6.60)
- moved C17 2.16 mm to (21.5, 4.57)
- moved R7 0.18 mm to (22.0, 31.4)
- moved R2 0.13 mm to (15.7, 8.51)
- flipped C18 to the bottom
- flipped C19 to the bottom
- renumbered J4 to J3
Connections:
- net CS renamed CS_BMS
- removed net DGND: IC1.P$6, J3.2
- new net CS_ADC: IC2.P$6, J3.7
- new net LDOIN: IC1.P$13, R35.P$2, R36.P$1
- new net N$8: C20.P$2, C21.P$2, IC2.P$1, V1.2
- net 3V3: now also C24.P$2, C25.P$2, IC2.P$9, J3.2, R1.P$1; no longer J3.3
- net 5V: now also C23.P$2, C26.P$2, C27.P$2, IC2.P$10, R36.P$2, V1.1; no longer IC1.P$13
- net AOUT: now also IC2.P$2; no longer J3.1
- net GND: now also C20.P$1, C21.P$1, C22.P$1, C23.P$1, C24.P$1, C25.P$1, C26.P$1, C27.P$1, IC1.P$6, IC2.P$3, IC2.P$4, IC2.P$5, J3.1, V1.3; no longer R1.P$1
- net SAMPL: now also J3.3; no longer J3.4
- net SCLK: now also IC2.P$8, J3.6; no longer J3.7
- net SDI: now also J3.5; no longer J3.6
- net SDO: now also IC2.P$7, J3.4; no longer J3.5
- net VP: now also C22.P$2, R35.P$1
Routing:
- net CS_ADC: track 0.00 -> 22.1 mm, vias 0 -> 1
- net 5V: track 3.58 -> 24.1 mm, vias 0 -> 2
- net 3V3: track 45.0 -> 62.9 mm, vias 1 -> 4
- net T3: track 23.2 -> 11.5 mm, vias 2 -> 0
- net DGND: track 9.07 -> 0.00 mm
- net T2: track 27.1 -> 18.6 mm, vias 2 -> 0
- net N$8: track 0.00 -> 8.28 mm
- net SCLK: track 15.5 -> 23.0 mm, vias 0 -> 1
- net SDO: track 12.5 -> 19.1 mm, vias 0 -> 1
- net LDOIN: track 0.00 -> 6.56 mm, vias 0 -> 1
- net T1: track 32.0 -> 25.7 mm, vias 1 -> 0
- net SAMPL: track 13.3 -> 8.45 mm
- net SDI: track 14.6 -> 10.8 mm
- net AOUT: track 11.7 -> 8.88 mm, vias 0 -> 1
- net N$40: track 7.01 -> 4.21 mm
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