File: Electronics/BMS/BMSMAX14921Breakout/BMSMAX14921Based.sch (EAGLE design)
At the start: 66 parts, among them IC1 MAX14921, J1 CONNECTOR_9PIN, J4 CONNECTOR_9PIN, J5 CONNECTOR_8PIN, J6 CONNECTOR_9PIN

Commit message: pcb spacer and breakoutoard over
Parts:
- added J2: CONNECTORJST2X9_2MM, MarkIIEaglelbr:CONNECTORJST2X9_2MM
Connections:
- net CV1: now also J2.P$2
- net CV10: now also J2.P$7
- net CV11: now also J2.P$6
- net CV12: now also J2.P$14
- net CV13: now also J2.P$13
- net CV14: now also J2.P$12
- net CV15: now also J2.P$11
- net CV2: now also J2.P$3
- net CV3: now also J2.P$4
- net CV4: now also J2.P$5
- net CV5: now also J2.P$15
- net CV6: now also J2.P$16
- net CV7: now also J2.P$17
- net CV8: now also J2.P$18
- net CV9: now also J2.P$8
- net GND: now also J2.P$1
- net VP: now also J2.P$10, J2.P$9

Commit message: updated Max14921 Breakout Board
Parts:
- removed J4: CONNECTOR_9PIN, lolomolo:CONNECTOR_9PIN
- added C20, C22, C25, C27: 1uF, lolomolo:CHIP_CAP0805
- added C21, C23, C24, C26: .1uF, lolomolo:CHIP_CAP0805
- added IC2: ADC141S626, MarkIIEaglelbr:ADC141S626
- added J3: CONNECTOR_9PIN, lolomolo:CONNECTOR_9PIN
- added R35, R36: 0, lolomolo:CHIP_RES0805
- added V1: (no value), MarkIIEaglelbr:REF3040
- C19: value 1uF -> .1uF
Connections:
- removed net CS: IC1.CS, J4.P$8, R2.P$1
- removed net DGND: IC1.DGND, J4.P$2
- new net CS_ADC: IC2.CS, J3.P$7
- new net CS_BMS: IC1.CS, J3.P$8, R2.P$1
- new net LDOIN: IC1.LDOIN, R35.P$1, R36.P$2
- new net N$8: C20.P$1, C21.P$1, IC2.VREF, V1.VOUT
- net 3V3: now also C24.P$1, C25.P$1, IC2.VIO, J3.P$2, R1.P$2; no longer J4.P$3
- net 5V: now also C23.P$1, C26.P$1, C27.P$1, IC2.VA, R36.P$1, V1.VIN; no longer IC1.LDOIN
- net AOUT: now also IC2.+IN; no longer J4.P$1
- net EN: now also J3.P$9; no longer J4.P$9
- net GND: now also C20.P$2, C21.P$2, C22.P$2, C23.P$2, C24.P$2, C25.P$2, C26.P$2, C27.P$2, IC1.DGND, IC2.-IN, IC2.GND, IC2.GND2, J3.P$1, V1.GND; no longer R1.P$2
- net SAMPL: now also J3.P$3; no longer J4.P$4
- net SCLK: now also IC2.SCLK, J3.P$6; no longer J4.P$7
- net SDI: now also J3.P$5; no longer J4.P$6
- net SDO: now also IC2.DOUT, J3.P$4; no longer J4.P$5
- net VP: now also C22.P$1, R35.P$2
Other:
- moved on the sheet: C19
